File: _saved_CMD.sch (KiCad schematic (older format))
At the start: 21 parts

Commit message: Added compoenents and made connections.
Parts:
- removed C?: CAP, symbol pspice:CAP
- removed U?: NE555P, digikey-footprints:DIP-8_W7.62mm, symbol dk_Clock-Timing-Programmable-Timers-and-Oscillators:NE555P
- added C?: CAP, symbol pspice:CAP
- added U?: 555, symbol dk_Clock-Timing-Programmable-Timers-and-Oscillators:555
- Q?: symbol Device:Q_NPN_BCE -> dk_Transistors-Bipolar-BJT-Single:2N3904
Connections:
- net labels added: Earth
- wire segments 0 -> 65

Commit message: Added foorprints, 3 footprints remaining.
Parts:
- added LS1: Speaker, symbol Device:Speaker
- added Volume-Control1: 200, Potentiometer_SMD:Potentiometer_ACP_CA14-VSMD_Vertical_Hole, symbol Device:R_POT
- 9V1: renamed from BT?; footprint (none) -> Connector:JWT_A3963_1x02_P3.96mm_Vertical
- C1, C2: renamed from C?; footprint (none) -> Capacitor_SMD:C_0805_2012Metric_Pad1.15x1.40mm_HandSolder
- C3: renamed from C?; value CP1 -> 10uF; footprint (none) -> Capacitor_SMD:C_0805_2012Metric_Pad1.15x1.40mm_HandSolder
- C4, C5: renamed from C?; value CAP -> 0.02uF; footprint (none) -> Capacitor_THT:CP_Axial_L10.0mm_D4.5mm_P15.00mm_Horizontal
- C6: renamed from C?; value CP1 -> 100uF; footprint (none) -> Capacitor_SMD:C_0805_2012Metric_Pad1.15x1.40mm_HandSolder
- LED1, LED2: renamed from D?; footprint (none) -> Diode_SMD:D_1206_3216Metric_Pad1.42x1.75mm_HandSolder
- Q1, Q2: renamed from Q?; footprint (none) -> Package_TO_SOT_THT:TO-92
- R1, R7: renamed from R?; value R -> 470; footprint (none) -> Resistor_SMD:R_0805_2012Metric_Pad1.15x1.40mm_HandSolder
- R2: renamed from R?; value R -> 1K; footprint (none) -> Resistor_SMD:R_0805_2012Metric_Pad1.15x1.40mm_HandSolder
- R3: renamed from R?; value R -> 68
- R4, R6: renamed from R?; value R -> 22K; footprint (none) -> Resistor_SMD:R_0805_2012Metric_Pad1.15x1.40mm_HandSolder
- R5: renamed from R?; value R -> 47K; footprint (none) -> Resistor_SMD:R_0805_2012Metric_Pad1.15x1.40mm_HandSolder
- R8, R9: renamed from R?; value R -> 10K; footprint (none) -> Resistor_SMD:R_0805_2012Metric_Pad1.15x1.40mm_HandSolder
- gave numbers to parts that had none: 1
Connections:
- wire segments 65 -> 80

Commit message: Started layout.
Parts:
- IC1: footprint (none) -> 555 timer:TI_National_Semiconductor-LMC555CMM-Level_A
- LS1: footprint (none) -> Connector:JWT_A3963_1x02_P3.96mm_Vertical
- R3: footprint (none) -> Resistor_SMD:R_0805_2012Metric_Pad1.15x1.40mm_HandSolder
Changed lines of the file:
@@
 F 0 "R3" V 5200 1100 50  0000 C CNN
 F 1 "68" V 5300 1100 50  0000 C CNN
-F 2 "" V 5380 1100 50  0001 C CNN
+F 2 "Resistor_SMD:R_0805_2012Metric_Pad1.15x1.40mm_HandSolder" V 5380 1100 50  0001 C CNN
 F 3 "~" H 5450 1100 50  0001 C CNN
 	1    5450 1100
@@
 F 0 "IC1" H 8600 3000 50  0000 L CNN
 F 1 "555" H 8600 2900 50  0000 L CNN
-F 2 "" H 9050 3600 50  0001 C CNN
+F 2 "555 timer:TI_National_Semiconductor-LMC555CMM-Level_A" H 9050 3600 50  0001 C CNN
 F 3 "" H 9050 3600 50  0001 C CNN
 	1    8300 3000
@@
 F 0 "LS1" H 9500 5500 50  0000 L CNN
 F 1 "Speaker" H 9500 5450 50  0000 L CNN
-F 2 "" H 9300 5300 50  0001 C CNN
+F 2 "Connector:JWT_A3963_1x02_P3.96mm_Vertical" H 9300 5300 50  0001 C CNN
 F 3 "~" H 9290 5450 50  0001 C CNN
 	1    9300 5500
@@
 Wire Wire Line
 	8400 6350 8400 6200
+$Comp
+L power:GNDD #PWR0103
+U 1 1 635573A4
+P 8400 6350
+F 0 "#PWR0103" H 8400 6100 50  0001 C CNN
+F 1 "GNDD" H 8450 6150 50  0000 C CNN
+F 2 "" H 8400 6350 50  0001 C CNN
+F 3 "" H 8400 6350 50  0001 C CNN
+	1    8400 6350
+	1    0    0    -1
+$EndComp
 $EndSCHEMATC
