File: CMD.kicad_pcb (KiCad board)
At the start: 2 copper layers, 23 parts, among them IC1 555, Q1 Q_NPN_BCE, Q2 Q_NPN_BCE

Commit message: Finished routing.
Parts:
- 9V1, LS1: footprint Connector:JWT_A3963_1x02_P3.96mm_Vertical -> Connector_Wire:SolderWirePad_1x02_P3.81mm_Drill1.2mm
- C4, C5: footprint Capacitor_THT:CP_Axial_L10.0mm_D4.5mm_P15.00mm_Horizontal -> Capacitor_SMD:C_1206_3216Metric
- moved IC1 40.4 mm to (168.3, 86.2)
- moved 9V1 40.3 mm to (174.3, 79.3), turned to 90 degrees
- moved LED1 39.2 mm to (127.5, 74.8), turned to 90 degrees
- moved C5 38.6 mm to (166.9, 80.7), turned to 180 degrees
- moved LS1 33.2 mm to (155.7, 74.5)
- moved Q2 30.9 mm to (133.3, 92.4), turned to 90 degrees
- moved R3 29.1 mm to (142.5, 77.5), turned to 180 degrees
- moved C6 27.9 mm to (166.9, 75.0)
- moved R2 27.2 mm to (137.1, 75.9), turned to 90 degrees
- moved R9 25.1 mm to (174.8, 88.1), turned to 90 degrees
- moved R6 24.1 mm to (167.2, 96.9)
- moved Q1 20.7 mm to (133.7, 84.1), turned to 90 degrees
- moved R5 16.4 mm to (160.3, 96.4)
- moved C4 13.8 mm to (142.1, 90.7)
- moved C1 13.3 mm to (139.1, 96.9)
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Routing:
- net Net-(9V1-Pad1): track 0.00 -> 88.2 mm
- net GNDD: track 0.00 -> 77.1 mm
- net Net-(C2-Pad1): track 0.00 -> 64.0 mm
- net Net-(C5-Pad1): track 0.00 -> 56.5 mm
- net Net-(R1-Pad1): track 0.00 -> 50.0 mm
- net Net-(C1-Pad2): track 0.00 -> 47.4 mm, vias 0 -> 1
- net Net-(IC1-Pad2): track 0.00 -> 38.1 mm
- net Net-(C4-Pad1): track 0.00 -> 35.0 mm, vias 0 -> 2
- net Net-(C2-Pad2): track 0.00 -> 23.3 mm
- net Net-(LED2-Pad1): track 0.00 -> 12.5 mm
- net Net-(C1-Pad1): track 0.00 -> 12.1 mm
- net Net-(C3-Pad2): track 0.00 -> 10.5 mm
- net Net-(LED1-Pad1): track 0.00 -> 8.53 mm
- net Net-(IC1-Pad5): track 0.00 -> 8.03 mm
- net Net-(C3-Pad1): track 0.00 -> 7.38 mm
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
Commit message: Replaced EARTH > GND, Replaced 555 Footprint.
Parts:
- IC1: footprint 555 timer:TI_National_Semiconductor-LMC555CMM-Level_A -> 555 Timer:Texas_Instruments-LMC555CMM_NOPB-Level_A
Changed lines of the file:
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@@
     (add_net "Net-(R1-Pad1)")
+  )
+  (module "555 Timer:Texas_Instruments-LMC555CMM_NOPB-Level_A" (layer F.Cu)
+    (at 168.326 86.233)
+    (fp_text reference IC1 (at -1.397 -0.096) (layer F.SilkS)
+      (effects (font (size 0.700001 0.700001) (thickness 0.15)) (justify left))
+    )
+    (fp_text value 555 (at 0 0) (layer F.SilkS)
+      (effects (font (size 1.27 1.27) (thickness 0.15)))
+    )
+    (fp_line (start 3.525 1.975001) (end 3.525 -1.974997) (layer F.CrtYd) (width 0.15))
+    (fp_line (start -3.525 1.975001) (end 3.525 1.975001) (layer F.CrtYd) (width 0.15))
+    (fp_line (start -3.525 -1.974997) (end -3.525 1.975001) (layer F.CrtYd) (width 0.15))
+    (fp_line (start 3.525 -1.974997) (end -3.525 -1.974997) (layer F.CrtYd) (width 0.15))
+    (fp_line (start 3.525 -1.974997) (end 3.525 -1.974997) (layer F.CrtYd) (width 0.15))
+    (fp_line (start -1.549999 1.549999) (end 1.550002 1.549999) (layer F.Fab) (width 0.1))
+    (fp_line (start -1.549999 -1.549999) (end 1.550002 -1.549999) (layer F.Fab) (width 0.1))
+    (fp_line (start 1.550002 1.549999) (end 1.550002 -1.549999) (layer F.Fab) (width 0.1))
+    (fp_line (start -1.549999 1.549999) (end -1.549999 -1.549999) (layer F.Fab) (width 0.1))
+    (fp_line (start -1.15 1.549999) (end 1.15 1.549999) (layer F.SilkS) (width 0.15))
+    (fp_line (start -1.15 -1.549999) (end 1.15 -1.549999) (layer F.SilkS) (width 0.15))
+    (fp_line (start 1.15 1.549999) (end 1.15 -1.549999) (layer F.SilkS) (width 0.15))
+    (fp_line (start -1.15 1.549999) (end -1.15 -1.549999) (layer F.SilkS) (width 0.15))
+    (fp_circle (center -2.324999 -1.799999) (end -2.199998 -1.799999) (layer F.SilkS) (width 0.249999))
+    (pad 1 smd roundrect (at -2.324999 -0.974999 270) (size 0.449999 1.549999) (layers F.Cu F.Paste F.Mask) (roundrect_rratio 0.4399965333)
+      (net 1 GNDD))
+    (pad 2 smd roundrect (at -2.324999 -0.324998 270) (size 0.449999 1.549999) (layers F.Cu F.Paste F.Mask) (roundrect_rratio 0.4399965333)
+      (net 13 "Net-(IC1-Pad2)"))
+    (pad 3 smd roundrect (at -2.324999 0.325001 270) (size 0.449999 1.549999) (layers F.Cu F.Paste F.Mask) (roundrect_rratio 0.4399965333)
+      (net 7 "Net-(C3-Pad1)"))
+    (pad 4 smd roundrect (at -2.324999 0.975002 270) (size 0.449999 1.549999) (layers F.Cu F.Paste F.Mask) (roundrect_rratio 0.4399965333)
+      (net 11 "Net-(C5-Pad1)"))
+    (pad 8 smd roundrect (at 2.325002 -0.974999 270) (size 0.449999 1.549999) (layers F.Cu F.Paste F.Mask) (roundrect_rratio 0.4399965333)
+      (net 11 "Net-(C5-Pad1)"))
+    (pad 7 smd roundrect (at 2.325002 -0.324998 270) (size 0.449999 1.549999) (layers F.Cu F.Paste F.Mask) (roundrect_rratio 0.4399965333)
+      (net 14 "Net-(IC1-Pad7)"))
+    (pad 6 smd roundrect (at 2.325002 0.325001 270) (size 0.449999 1.549999) (layers F.Cu F.Paste F.Mask) (roundrect_rratio 0.4399965333)
+      (net 13 "Net-(IC1-Pad2)"))
+    (pad 5 smd roundrect (at 2.325002 0.975002 270) (size 0.449999 1.549999) (layers F.Cu F.Paste F.Mask) (roundrect_rratio 0.4399965333)
+      (net 12 "Net-(IC1-Pad5)"))
   )
   (module Capacitor_SMD:C_1206_3216Metric (layer F.Cu)
@@
     )
   )
-  (module "555 timer:TI_National_Semiconductor-LMC555CMM-Level_A" (layer F.Cu)
-    (at 168.326 86.233)
-    (fp_text reference IC1 (at -1.397 -0.096) (layer F.SilkS)
-      (effects (font (size 0.700001 0.700001) (thickness 0.15)) (justify left))
-    )
-    (fp_text value 555 (at 0 0) (layer F.SilkS)
-      (effects (font (size 1.27 1.27) (thickness 0.15)))
-    )
-    (fp_circle (center -2.324999 -1.799999) (end -2.199998 -1.799999) (layer F.SilkS) (width 0.249999))
-    (fp_line (start -1.15 1.549999) (end -1.15 -1.549999) (layer F.SilkS) (width 0.15))
-    (fp_line (start 1.15 1.549999) (end 1.15 -1.549999) (layer F.SilkS) (width 0.15))
-    (fp_line (start -1.15 -1.549999) (end 1.15 -1.549999) (layer F.SilkS) (width 0.15))
-    (fp_line (start -1.15 1.549999) (end 1.15 1.549999) (layer F.SilkS) (width 0.15))
-    (fp_line (start -1.549999 1.549999) (end -1.549999 -1.549999) (layer F.Fab) (width 0.1))
-    (fp_line (start 1.550002 1.549999) (end 1.550002 -1.549999) (layer F.Fab) (width 0.1))
-    (fp_line (start -1.549999 -1.549999) (end 1.550002 -1.549999) (layer F.Fab) (width 0.1))
-    (fp_line (start -1.549999 1.549999) (end 1.550002 1.549999) (layer F.Fab) (width 0.1))
-    (fp_line (start 3.525 -1.974997) (end 3.525 -1.974997) (layer F.CrtYd) (width 0.15))
-    (fp_line (start 3.525 -1.974997) (end -3.525 -1.974997) (layer F.CrtYd) (width 0.15))
-    (fp_line (start -3.525 -1.974997) (end -3.525 1.975001) (layer F.CrtYd) (width 0.15))
-    (fp_line (start -3.525 1.975001) (end 3.525 1.975001) (layer F.CrtYd) (width 0.15))
-    (fp_line (start 3.525 1.975001) (end 3.525 -1.974997) (layer F.CrtYd) (width 0.15))
-    (pad 5 smd roundrect (at 2.325002 0.975002 270) (size 0.449999 1.549999) (layers F.Cu F.Paste F.Mask) (roundrect_rratio 0.4399965333)
-      (net 12 "Net-(IC1-Pad5)"))
-    (pad 6 smd roundrect (at 2.325002 0.325001 270) (size 0.449999 1.549999) (layers F.Cu F.Paste F.Mask) (roundrect_rratio 0.4399965333)
-      (net 13 "Net-(IC1-Pad2)"))
-    (pad 7 smd roundrect (at 2.325002 -0.324998 270) (size 0.449999 1.549999) (layers F.Cu F.Paste F.Mask) (roundrect_rratio 0.4399965333)
-      (net 14 "Net-(IC1-Pad7)"))
-    (pad 8 smd roundrect (at 2.325002 -0.974999 270) (size 0.449999 1.549999) (layers F.Cu F.Paste F.Mask) (roundrect_rratio 0.4399965333)
-      (net 11 "Net-(C5-Pad1)"))
-    (pad 4 smd roundrect (at -2.324999 0.975002 270) (size 0.449999 1.549999) (layers F.Cu F.Paste F.Mask) (roundrect_rratio 0.4399965333)
-      (net 11 "Net-(C5-Pad1)"))
-    (pad 3 smd roundrect (at -2.324999 0.325001 270) (size 0.449999 1.549999) (layers F.Cu F.Paste F.Mask) (roundrect_rratio 0.4399965333)
-      (net 7 "Net-(C3-Pad1)"))
-    (pad 2 smd roundrect (at -2.324999 -0.324998 270) (size 0.449999 1.549999) (layers F.Cu F.Paste F.Mask) (roundrect_rratio 0.4399965333)
-      (net 13 "Net-(IC1-Pad2)"))
-    (pad 1 smd roundrect (at -2.324999 -0.974999 270) (size 0.449999 1.549999) (layers F.Cu F.Paste F.Mask) (roundrect_rratio 0.4399965333)
-      (net 1 GNDD))
-  )
   (module Diode_SMD:D_1206_3216Metric_Pad1.42x1.75mm_HandSolder (layer F.Cu)
