File: CMD.sch (KiCad schematic (older format))
At the start: 15 parts

Commit message: Added foorprints, 3 footprints remaining.
Parts:
- added C3: 10uF, Capacitor_SMD:C_0805_2012Metric_Pad1.15x1.40mm_HandSolder, symbol Device:CP1
- added C4, C5: 0.02uF, Capacitor_THT:CP_Axial_L10.0mm_D4.5mm_P15.00mm_Horizontal, symbol pspice:CAP
- added IC1: 555, symbol dk_Clock-Timing-Programmable-Timers-and-Oscillators:555
- added LS?: Speaker, symbol Device:Speaker
- added R5: 47K, Resistor_SMD:R_0805_2012Metric_Pad1.15x1.40mm_HandSolder, symbol Device:R
- added R9: 10K, Resistor_SMD:R_0805_2012Metric_Pad1.15x1.40mm_HandSolder, symbol Device:R
- added Volume-Control: 200, Potentiometer_SMD:Potentiometer_ACP_CA14-VSMD_Vertical_Hole, symbol Device:R_POT
- 9V: renamed from BT?; footprint (none) -> Connector:JWT_A3963_1x02_P3.96mm_Vertical
- C1, C2: renamed from C?; footprint (none) -> Capacitor_SMD:C_0805_2012Metric_Pad1.15x1.40mm_HandSolder
- C6: renamed from C?; value CP1 -> 100uF; footprint (none) -> Capacitor_SMD:C_0805_2012Metric_Pad1.15x1.40mm_HandSolder
- LED1, LED2: renamed from D?; footprint (none) -> Diode_SMD:D_1206_3216Metric_Pad1.42x1.75mm_HandSolder
- Q1: renamed from Q?; footprint (none) -> Package_TO_SOT_THT:TO-92; symbol Device:Q_NPN_BCE -> dk_Transistors-Bipolar-BJT-Single:2N3904
- Q2: renamed from Q?; footprint (none) -> Package_TO_SOT_THT:TO-92
- R1, R7: renamed from R?; value R -> 470; footprint (none) -> Resistor_SMD:R_0805_2012Metric_Pad1.15x1.40mm_HandSolder
- R2: renamed from R?; value R -> 1K; footprint (none) -> Resistor_SMD:R_0805_2012Metric_Pad1.15x1.40mm_HandSolder
- R3: renamed from R?; value R -> 68
- R4, R6: renamed from R?; value R -> 22K; footprint (none) -> Resistor_SMD:R_0805_2012Metric_Pad1.15x1.40mm_HandSolder
- R8: renamed from R?; value R -> 10K; footprint (none) -> Resistor_SMD:R_0805_2012Metric_Pad1.15x1.40mm_HandSolder
Connections:
- net labels added: Earth
- wire segments 0 -> 80

Commit message: Started layout.
Parts:
- gave numbers to parts that had none: 1
- renumbered 9V to 9V1, Volume-Control to Volume-Control1
Connections:
- net labels added: GNDD
Changed lines of the file:
@@
 $EndDescr
 $Comp
-L Device:Battery 9V
+L Device:Battery 9V1
 U 1 1 634C5E09
 P 1000 3150
-F 0 "9V" H 1150 3200 50  0000 L CNN
+F 0 "9V1" H 1150 3200 50  0000 L CNN
 F 1 "Battery" H 1150 3150 50  0000 L CNN
 F 2 "Connector:JWT_A3963_1x02_P3.96mm_Vertical" V 1000 3210 50  0001 C CNN
@@
 	9950 2500 9950 2700
 $Comp
-L power:Earth #PWR?
+L power:Earth #PWR0101
 U 1 1 6351710E
 P 9950 3550
-F 0 "#PWR?" H 9950 3300 50  0001 C CNN
+F 0 "#PWR0101" H 9950 3300 50  0001 C CNN
 F 1 "Earth" H 9950 3400 50  0001 C CNN
 F 2 "" H 9950 3550 50  0001 C CNN
@@
 Connection ~ 8400 2750
 $Comp
-L Device:R_POT Volume-Control
+L Device:R_POT Volume-Control1
 U 1 1 63536E41
 P 8400 5500
-F 0 "Volume-Control" H 8300 5550 50  0000 R CNN
+F 0 "Volume-Control1" H 8300 5550 50  0000 R CNN
 F 1 "200" H 8300 5500 50  0000 R CNN
 F 2 "Potentiometer_SMD:Potentiometer_ACP_CA14-VSMD_Vertical_Hole" H 8400 5500 50  0001 C CNN
@@
 	8400 5350 8400 5050
 $Comp
-L Device:Speaker LS?
+L Device:Speaker LS1
 U 1 1 63539103
 P 9300 5500
-F 0 "LS?" H 9500 5500 50  0000 L CNN
+F 0 "LS1" H 9500 5500 50  0000 L CNN
 F 1 "Speaker" H 9500 5450 50  0000 L CNN
 F 2 "" H 9300 5300 50  0001 C CNN
@@
 	8800 6200 8400 6200
 Connection ~ 8400 6200
-Wire Wire Line
-	8400 6200 8400 6350
-$Comp
-L power:Earth #PWR?
-U 1 1 6353DD53
-P 8400 6350
-F 0 "#PWR?" H 8400 6100 50  0001 C CNN
-F 1 "Earth" H 8400 6200 50  0001 C CNN
-F 2 "" H 8400 6350 50  0001 C CNN
-F 3 "~" H 8400 6350 50  0001 C CNN
-	1    8400 6350
-	1    0    0    -1
-$EndComp
 Connection ~ 4950 6200
 Connection ~ 2800 6200
-$Comp
-L power:Earth #PWR?
-U 1 1 63540573
-P 4950 6400
-F 0 "#PWR?" H 4950 6150 50  0001 C CNN
-F 1 "Earth" H 4950 6250 50  0001 C CNN
-F 2 "" H 4950 6400 50  0001 C CNN
-F 3 "~" H 4950 6400 50  0001 C CNN
-	1    4950 6400
-	1    0    0    -1
-$EndComp
-Wire Wire Line
-	4950 6400 4950 6200
 Wire Wire Line
 	1900 4000 1900 6200
@@
 Wire Wire Line
 	1900 6200 2800 6200
+$Comp
+L power:GNDD #PWR0102
+U 1 1 6354FCB2
+P 2800 6500
+F 0 "#PWR0102" H 2800 6250 50  0001 C CNN
+F 1 "GNDD" H 2850 6300 50  0000 C CNN
+F 2 "" H 2800 6500 50  0001 C CNN
+F 3 "" H 2800 6500 50  0001 C CNN
+	1    2800 6500
+	1    0    0    -1
+$EndComp
+Wire Wire Line
+	2800 6500 2800 6200
+Wire Wire Line
+	8400 6350 8400 6200
 $EndSCHEMATC

Commit message: Replaced EARTH > GND, Replaced 555 Footprint.
Parts:
- IC1: footprint (none) -> 555 timer:TI_National_Semiconductor-LMC555CMM-Level_A
- LS1: footprint (none) -> Connector:JWT_A3963_1x02_P3.96mm_Vertical
- R3: footprint (none) -> Resistor_SMD:R_0805_2012Metric_Pad1.15x1.40mm_HandSolder
Connections:
- net labels removed: Earth
Changed lines of the file:
@@
 EESchema Schematic File Version 4
+LIBS:CMD-cache
 EELAYER 26 0
 EELAYER END
@@
 F 0 "R3" V 5200 1100 50  0000 C CNN
 F 1 "68" V 5300 1100 50  0000 C CNN
-F 2 "" V 5380 1100 50  0001 C CNN
+F 2 "Resistor_SMD:R_0805_2012Metric_Pad1.15x1.40mm_HandSolder" V 5380 1100 50  0001 C CNN
 F 3 "~" H 5450 1100 50  0001 C CNN
 	1    5450 1100
@@
 F 0 "IC1" H 8600 3000 50  0000 L CNN
 F 1 "555" H 8600 2900 50  0000 L CNN
-F 2 "" H 9050 3600 50  0001 C CNN
+F 2 "555 timer:TI_National_Semiconductor-LMC555CMM-Level_A" H 9050 3600 50  0001 C CNN
 F 3 "" H 9050 3600 50  0001 C CNN
 	1    8300 3000
@@
 Wire Wire Line
 	9950 2500 9950 2700
-$Comp
-L power:Earth #PWR0101
-U 1 1 6351710E
-P 9950 3550
-F 0 "#PWR0101" H 9950 3300 50  0001 C CNN
-F 1 "Earth" H 9950 3400 50  0001 C CNN
-F 2 "" H 9950 3550 50  0001 C CNN
-F 3 "~" H 9950 3550 50  0001 C CNN
-	1    9950 3550
-	1    0    0    -1
-$EndComp
-Wire Wire Line
-	9950 3550 9950 3200
 Wire Wire Line
 	8950 1100 7300 1100
@@
 	8200 3600 7300 3600
 Connection ~ 7300 3600
-Wire Wire Line
-	7300 3600 7300 6200
 Wire Wire Line
 	7050 2750 7050 3750
@@
 F 0 "LS1" H 9500 5500 50  0000 L CNN
 F 1 "Speaker" H 9500 5450 50  0000 L CNN
-F 2 "" H 9300 5300 50  0001 C CNN
+F 2 "Connector:JWT_A3963_1x02_P3.96mm_Vertical" H 9300 5300 50  0001 C CNN
 F 3 "~" H 9290 5450 50  0001 C CNN
 	1    9300 5500
@@
 Wire Wire Line
 	2800 6500 2800 6200
-Wire Wire Line
-	8400 6350 8400 6200
+$Comp
+L power:GNDD #PWR0103
+U 1 1 635573A4
+P 7300 6400
+F 0 "#PWR0103" H 7300 6150 50  0001 C CNN
+F 1 "GNDD" H 7350 6200 50  0000 C CNN
+F 2 "" H 7300 6400 50  0001 C CNN
+F 3 "" H 7300 6400 50  0001 C CNN
+	1    7300 6400
+	1    0    0    -1
+$EndComp
+Connection ~ 7300 6050
+Wire Wire Line
+	7300 6050 7300 6200
+Wire Wire Line
+	7300 6200 7300 6400
+Wire Wire Line
+	7300 3600 7300 6200
 $EndSCHEMATC
